Commit message: completion of urdf file to add the robot arm to the

File: src/wheel_robot/urdf/robot1_with_arm.urdf (robot description, URDF)
Before this commit: robot robot1, 10 links, 9 joints
Links:
- added link left_gripper
- added link left_tip; visual mesh filename=package://wheel_robot/meshes/gripper_v0/l_finger_tip.stl
Joints:
- added joint left_gripper_joint: type revolute, parent arm_2, child left_gripper, origin xyz=0.06 0 0.4 rpy=0 -1.57 0, axis 0 0 1, limit lower=0 upper=0.548 effort=1000 velocity=0.5
- added joint left_tip_joint: type fixed, parent left_gripper, child left_tip
